File: kicad_project/electronic_load.sch (KiCad schematic (older format))
At the start: 0 parts

Commit message: doing stuff
Changed lines of the file:
@@
 $Descr A4 11693 8268
 encoding utf-8
-Sheet 1 4
+Sheet 1 5
 Title ""
 Date ""
@@
 F1 "file5CACBC99.sch" 50
 $EndSheet
+$Sheet
+S 5850 3900 500  150
+U 5CAD5603
+F0 "monitor_outputs" 50
+F1 "file5CAD5602.sch" 50
+$EndSheet
 $EndSCHEMATC
