File: kicad_project/file5CACB7A8.sch (KiCad schematic (older format))
At the start: 13 parts

Commit message: doing stuff
Parts:
- removed U?: OPA656, Package_TO_SOT_SMD:SOT-23-5, symbol Amplifier_Operational:OP179GRT
Changed lines of the file:
@@
 $Descr A4 11693 8268
 encoding utf-8
-Sheet 2 4
+Sheet 2 5
 Title ""
 Date ""
@@
 Gate\nSource\nGround\n(Kelvin connections)
 Wire Wire Line
-	6500 4450 6800 4450
+	4400 5100 4700 5100
 $Comp
 L Device:R R?
 U 1 1 5CAE519B
-P 5550 4850
-F 0 "R?" H 5480 4804 50  0000 R CNN
-F 1 "18k" H 5480 4895 50  0000 R CNN
-F 2 "" V 5480 4850 50  0001 C CNN
-F 3 "~" H 5550 4850 50  0001 C CNN
-	1    5550 4850
+P 3450 5500
+F 0 "R?" H 3380 5454 50  0000 R CNN
+F 1 "18k" H 3380 5545 50  0000 R CNN
+F 2 "" V 3380 5500 50  0001 C CNN
+F 3 "~" H 3450 5500 50  0001 C CNN
+	1    3450 5500
 	-1   0    0    1
 $EndComp
@@
 L Device:R R?
 U 1 1 5CAE51A2
-P 5550 5350
-F 0 "R?" H 5480 5304 50  0000 R CNN
-F 1 "2k" H 5480 5395 50  0000 R CNN
-F 2 "" V 5480 5350 50  0001 C CNN
-F 3 "~" H 5550 5350 50  0001 C CNN
-	1    5550 5350
+P 3450 6000
+F 0 "R?" H 3380 5954 50  0000 R CNN
+F 1 "2k" H 3380 6045 50  0000 R CNN
+F 2 "" V 3380 6000 50  0001 C CNN
+F 3 "~" H 3450 6000 50  0001 C CNN
+	1    3450 6000
 	-1   0    0    1
 $EndComp
@@
 L power:GND #PWR?
 U 1 1 5CAE51A9
-P 5550 5600
-F 0 "#PWR?" H 5550 5350 50  0001 C CNN
-F 1 "GND" H 5555 5427 50  0000 C CNN
-F 2 "" H 5550 5600 50  0001 C CNN
-F 3 "" H 5550 5600 50  0001 C CNN
-	1    5550 5600
-	1    0    0    -1
-$EndComp
-Wire Wire Line
-	5550 5600 5550 5500
-Wire Wire Line
-	5550 5200 5550 5100
-Wire Wire Line
-	5550 4700 5550 4350
-Wire Wire Line
-	5550 4350 5900 4350
-Wire Wire Line
-	5550 5100 6800 5100
-Wire Wire Line
-	6800 5100 6800 4450
-Connection ~ 5550 5100
-Wire Wire Line
-	5550 5100 5550 5000
+P 3450 6250
+F 0 "#PWR?" H 3450 6000 50  0001 C CNN
+F 1 "GND" H 3455 6077 50  0000 C CNN
+F 2 "" H 3450 6250 50  0001 C CNN
+F 3 "" H 3450 6250 50  0001 C CNN
+	1    3450 6250
+	1    0    0    -1
+$EndComp
+Wire Wire Line
+	3450 6250 3450 6150
+Wire Wire Line
+	3450 5850 3450 5750
+Wire Wire Line
+	3450 5350 3450 5000
+Wire Wire Line
+	3450 5000 3800 5000
+Wire Wire Line
+	3450 5750 4700 5750
+Wire Wire Line
+	4700 5750 4700 5100
+Connection ~ 3450 5750
+Wire Wire Line
+	3450 5750 3450 5650
 $Comp
 L power:GND #PWR?
 U 1 1 5CAE51B8
-P 4650 4500
-F 0 "#PWR?" H 4650 4250 50  0001 C CNN
-F 1 "GND" H 4655 4327 50  0000 C CNN
-F 2 "" H 4650 4500 50  0001 C CNN
-F 3 "" H 4650 4500 50  0001 C CNN
-	1    4650 4500
-	1    0    0    -1
-$EndComp
-Wire Wire Line
-	4450 4450 4650 4450
-Wire Wire Line
-	4650 4450 4650 4500
+P 2550 5150
+F 0 "#PWR?" H 2550 4900 50  0001 C CNN
+F 1 "GND" H 2555 4977 50  0000 C CNN
+F 2 "" H 2550 5150 50  0001 C CNN
+F 3 "" H 2550 5150 50  0001 C CNN
+	1    2550 5150
+	1    0    0    -1
+$EndComp
+Wire Wire Line
+	2350 5100 2550 5100
+Wire Wire Line
+	2550 5100 2550 5150
 $Comp
 L Connector_Generic:Conn_01x02 J?
 U 1 1 5CAE51C0
-P 4250 4450
-F 0 "J?" H 4170 4125 50  0000 C CNN
-F 1 "Conn_01x02" H 4170 4216 50  0000 C CNN
-F 2 "" H 4250 4450 50  0001 C CNN
-F 3 "~" H 4250 4450 50  0001 C CNN
-	1    4250 4450
+P 2150 5100
+F 0 "J?" H 2070 4775 50  0000 C CNN
+F 1 "Conn_01x02" H 2070 4866 50  0000 C CNN
+F 2 "" H 2150 5100 50  0001 C CNN
+F 3 "~" H 2150 5100 50  0001 C CNN
+	1    2150 5100
 	-1   0    0    1
 $EndComp
@@
 L Device:R R?
 U 1 1 5CAE51C7
-P 5050 4350
+P 2950 5000
 AR Path="/5CAE51C7" Ref="R?"  Part="1"
 AR Path="/5CACB7A9/5CAE51C7" Ref="R?"  Part="1"
-F 0 "R?" V 4843 4350 50  0000 C CNN
-F 1 "50" V 4934 4350 50  0000 C CNN
-F 2 "" V 4980 4350 50  0001 C CNN
-F 3 "~" H 5050 4350 50  0001 C CNN
-	1    5050 4350
+F 0 "R?" V 2743 5000 50  0000 C CNN
+F 1 "50" V 2834 5000 50  0000 C CNN
+F 2 "" V 2880 5000 50  0001 C CNN
+F 3 "~" H 2950 5000 50  0001 C CNN
+	1    2950 5000
 	0    1    1    0
 $EndComp
 Wire Wire Line
-	5200 4350 5550 4350
-Connection ~ 5550 4350
-Text GLabel 7100 4250 2    50   Input ~ 0
+	3100 5000 3450 5000
+Connection ~ 3450 5000
+Text GLabel 5000 4900 2    50   Input ~ 0
 Isense
 Wire Wire Line
-	7100 4250 6500 4250
-Text Notes 5250 3750 0    50   ~ 0
+	5000 4900 4400 4900
+Text Notes 3150 4400 0    50   ~ 0
 Current sense amp\nfor 50 ohm terminated o-scope
 Text Notes 6750 1150 0    50   ~ 0
 FIXME\nadd a shutdown mechanism\nfuse?\npulldown resistor
 Wire Wire Line
-	4450 4350 4900 4350
-$Comp
-L Amplifier_Operational:OP179GRT U?
-U 1 1 5CA330E5
-P 7100 5800
-F 0 "U?" H 7441 5846 50  0000 L CNN
-F 1 "OPA656" H 7441 5755 50  0000 L CNN
-F 2 "Package_TO_SOT_SMD:SOT-23-5" H 7100 5800 50  0001 C CNN
-F 3 "" H 7100 6000 50  0001 C CNN
-	1    7100 5800
-	1    0    0    -1
-$EndComp
-Text Notes 8400 4800 0    50   ~ 0
+	2350 5000 2800 5000
+Text Notes 6300 5450 0    50   ~ 0
 fixme opa2810
 $EndSCHEMATC
