File: kicad_project/file5CACB7D0.sch (KiCad schematic (older format))
At the start: 20 parts

Commit message: doing stuff
Parts:
- added J?: Conn_01x03, symbol Connector_Generic:Conn_01x03
- C?: value 0.1u -> 1u
- R?: value 15k -> 2.7k
Connections:
- wire segments 69 -> 74
Other:
- note added: "1MEG pot for frequency adjust 500 hz to 1hz"
- note added: "2.5v reference"
- note added: "DAC"
- moved on the sheet: U?B
Changed lines of the file:
@@
 $Descr A3 16535 11693
 encoding utf-8
-Sheet 3 4
+Sheet 3 5
 Title ""
 Date ""
@@
 AR Path="/5CACB7D1/5CAD0311" Ref="C?"  Part="1"
 F 0 "C?" H 5015 1446 50  0000 L CNN
-F 1 "0.1u" H 5015 1355 50  0000 L CNN
+F 1 "1u" H 5015 1355 50  0000 L CNN
 F 2 "" H 4938 1250 50  0001 C CNN
 F 3 "~" H 4900 1400 50  0001 C CNN
@@
 L Device:R R?
 U 1 1 5CAD031C
-P 5750 1200
+P 5650 1200
 AR Path="/5CAD031C" Ref="R?"  Part="1"
 AR Path="/5CACB7D1/5CAD031C" Ref="R?"  Part="1"
-F 0 "R?" V 5543 1200 50  0000 C CNN
-F 1 "15k" V 5634 1200 50  0000 C CNN
-F 2 "" V 5680 1200 50  0001 C CNN
-F 3 "~" H 5750 1200 50  0001 C CNN
-	1    5750 1200
+F 0 "R?" V 5443 1200 50  0000 C CNN
+F 1 "2.7k" V 5534 1200 50  0000 C CNN
+F 2 "" V 5580 1200 50  0001 C CNN
+F 3 "~" H 5650 1200 50  0001 C CNN
+	1    5650 1200
 	0    1    1    0
 $EndComp
 Wire Wire Line
-	5600 1200 5350 1200
+	5500 1200 5350 1200
 Connection ~ 5350 1200
-Wire Wire Line
-	5900 1200 6750 1200
 Wire Wire Line
 	6750 1200 6750 1950
@@
 L Amplifier_Operational:TL072 U?
 U 2 1 5CAD03E9
-P 8900 6750
+P 9700 6850
 AR Path="/5CAD03E9" Ref="U?"  Part="2"
 AR Path="/5CACB7D1/5CAD03E9" Ref="U?"  Part="2"
-F 0 "U?" H 9000 6500 50  0000 C CNN
-F 1 "TL072" H 9000 6600 50  0000 C CNN
-F 2 "" H 8900 6750 50  0001 C CNN
-F 3 "http://www.ti.com/lit/ds/symlink/tl071.pdf" H 8900 6750 50  0001 C CNN
-	2    8900 6750
-	1    0    0    -1
-$EndComp
-Text GLabel 9900 6750 2    50   Input ~ 0
+F 0 "U?" H 9800 6600 50  0000 C CNN
+F 1 "TL072" H 9800 6700 50  0000 C CNN
+F 2 "" H 9700 6850 50  0001 C CNN
+F 3 "http://www.ti.com/lit/ds/symlink/tl071.pdf" H 9700 6850 50  0001 C CNN
+	2    9700 6850
+	1    0    0    -1
+$EndComp
+Text GLabel 10700 6850 2    50   Input ~ 0
 Vref_DAC
 Wire Wire Line
-	9900 6750 9500 6750
+	10700 6850 10300 6850
 Text GLabel 14300 6050 0    50   Input ~ 0
 Vref_DAC
@@
 L Device:R R?
 U 1 1 5CAD0404
-P 9500 7150
+P 10300 7250
 AR Path="/5CAD0404" Ref="R?"  Part="1"
 AR Path="/5CACB7D1/5CAD0404" Ref="R?"  Part="1"
-F 0 "R?" H 9430 7104 50  0000 R CNN
-F 1 "10k" H 9430 7195 50  0000 R CNN
-F 2 "" V 9430 7150 50  0001 C CNN
-F 3 "~" H 9500 7150 50  0001 C CNN
-	1    9500 7150
+F 0 "R?" H 10230 7204 50  0000 R CNN
+F 1 "10k" H 10230 7295 50  0000 R CNN
+F 2 "" V 10230 7250 50  0001 C CNN
+F 3 "~" H 10300 7250 50  0001 C CNN
+	1    10300 7250
 	-1   0    0    1
 $EndComp
@@
 L Device:R R?
 U 1 1 5CAD040B
-P 9500 7650
+P 10300 7750
 AR Path="/5CAD040B" Ref="R?"  Part="1"
 AR Path="/5CACB7D1/5CAD040B" Ref="R?"  Part="1"
-F 0 "R?" H 9430 7604 50  0000 R CNN
-F 1 "10k" H 9430 7695 50  0000 R CNN
-F 2 "" V 9430 7650 50  0001 C CNN
-F 3 "~" H 9500 7650 50  0001 C CNN
-	1    9500 7650
+F 0 "R?" H 10230 7704 50  0000 R CNN
+F 1 "10k" H 10230 7795 50  0000 R CNN
+F 2 "" V 10230 7750 50  0001 C CNN
+F 3 "~" H 10300 7750 50  0001 C CNN
+	1    10300 7750
 	-1   0    0    1
 $EndComp
 Wire Wire Line
-	9500 7000 9500 6750
-Connection ~ 9500 6750
-Wire Wire Line
-	9500 6750 9200 6750
-Wire Wire Line
-	9500 7300 9500 7400
-Wire Wire Line
-	9500 7400 8300 7400
-Wire Wire Line
-	8300 7400 8300 6850
-Wire Wire Line
-	8300 6850 8600 6850
-Connection ~ 9500 7400
-Wire Wire Line
-	9500 7400 9500 7500
+	10300 7100 10300 6850
+Connection ~ 10300 6850
+Wire Wire Line
+	10300 6850 10000 6850
+Wire Wire Line
+	10300 7400 10300 7500
+Wire Wire Line
+	10300 7500 9100 7500
+Wire Wire Line
+	9100 7500 9100 6950
+Wire Wire Line
+	9100 6950 9400 6950
+Connection ~ 10300 7500
+Wire Wire Line
+	10300 7500 10300 7600
 $Comp
 L power:GND #PWR?
 U 1 1 5CAD041B
-P 9500 7900
+P 10300 8000
 AR Path="/5CAD041B" Ref="#PWR?"  Part="1"
 AR Path="/5CACB7D1/5CAD041B" Ref="#PWR?"  Part="1"
-F 0 "#PWR?" H 9500 7650 50  0001 C CNN
-F 1 "GND" H 9505 7727 50  0000 C CNN
-F 2 "" H 9500 7900 50  0001 C CNN
-F 3 "" H 9500 7900 50  0001 C CNN
-	1    9500 7900
-	1    0    0    -1
-$EndComp
-Wire Wire Line
-	9500 7900 9500 7800
+F 0 "#PWR?" H 10300 7750 50  0001 C CNN
+F 1 "GND" H 10305 7827 50  0000 C CNN
+F 2 "" H 10300 8000 50  0001 C CNN
+F 3 "" H 10300 8000 50  0001 C CNN
+	1    10300 8000
+	1    0    0    -1
+$EndComp
+Wire Wire Line
+	10300 8000 10300 7900
 Text Notes 9700 3750 0    50   ~ 0
 10k pot
 Text Notes 7250 2500 0    50   ~ 0
 10k pot
-Text Notes 5400 700  0    50   ~ 0
+Text Notes 4800 650  0    50   ~ 0
 500hz oscillator
-Text GLabel 7550 6650 0    50   Input ~ 0
+Text GLabel 8350 6750 0    50   Input ~ 0
 DAC_OUT
 Wire Wire Line
-	7550 6650 8600 6650
-Text Notes 8500 6200 0    50   ~ 0
+	8350 6750 9400 6750
+Text Notes 9300 6300 0    50   ~ 0
 DAC Amplifier 2.5v to 5v
 Text Notes 7450 1200 0    50   ~ 0
@@
 Text Notes 10850 1000 0    50   ~ 0
 summing amplifier
+$Comp
+L Connector_Generic:Conn_01x03 J?
+U 1 1 5CAC8914
+P 6300 900
+AR Path="/5CAC8914" Ref="J?"  Part="1"
+AR Path="/5CACB7D1/5CAC8914" Ref="J?"  Part="1"
+F 0 "J?" V 6300 1150 50  0000 C CNN
+F 1 "Conn_01x03" V 6450 1050 50  0000 C CNN
+F 2 "" H 6300 900 50  0001 C CNN
+F 3 "~" H 6300 900 50  0001 C CNN
+	1    6300 900
+	0    1    -1   0
+$EndComp
+Wire Wire Line
+	6200 1100 6200 1200
+Wire Wire Line
+	6200 1200 5800 1200
+Wire Wire Line
+	6400 1100 6400 1200
+Wire Wire Line
+	6400 1200 6750 1200
+Wire Wire Line
+	6300 1100 6300 1200
+Wire Wire Line
+	6300 1200 6200 1200
+Connection ~ 6200 1200
+Text Notes 5900 650  0    50   ~ 0
+1MEG pot for frequency adjust 500 hz to 1hz
+Wire Notes Line
+	12000 5600 12000 9200
+Wire Notes Line
+	12000 9200 1100 9200
+Wire Notes Line
+	1100 9200 1100 5600
+Wire Notes Line
+	1100 5600 12000 5600
+Text Notes 3300 6100 0    50   ~ 0
+DAC
+Wire Notes Line
+	13550 4450 13550 6400
+Wire Notes Line
+	13550 6400 15700 6400
+Wire Notes Line
+	15700 6400 15700 4450
+Wire Notes Line
+	15700 4450 13550 4450
+Wire Notes Line
+	2400 500  13100 500
+Wire Notes Line
+	13100 500  13100 4700
+Wire Notes Line
+	13100 4700 2400 4700
+Wire Notes Line
+	2400 4700 2400 500
+Wire Notes Line
+	13550 1050 13550 3750
+Wire Notes Line
+	13550 3750 15450 3750
+Wire Notes Line
+	15450 3750 15450 1050
+Wire Notes Line
+	15450 1050 13550 1050
+Text Notes 14250 1400 0    50   ~ 0
+2.5v reference
 $EndSCHEMATC
