File: kicad_project/file5CACBC99.sch (KiCad schematic (older format))
At the start: 8 parts

Commit message: doing stuff
Parts:
- added R?: 1.3k, symbol Device:R
Connections:
- net labels added: +3V3, Vin
- net labels removed: VCC
- wire segments 26 -> 28
Other:
- moved on the sheet: U?A, U?B
